File: AnalogPIDController/AnalogPIDController.kicad_pcb (KiCad board)
At the start: 2 copper layers, 51 parts, among them Q1 Q_NPN, U1 TL082, U2 TL084

Commit message: placing (w/o routing)
Parts:
- moved R3 151.6 mm to (175.5, 41.7), turned to 90 degrees
- moved R15 146.6 mm to (169.5, 57.9), turned to -90 degrees
- moved TP3 141.5 mm to (179.5, 46.5)
- moved R1 140.6 mm to (165.0, 24.4), turned to -90 degrees
- moved R16 140.6 mm to (163.6, 63.0), turned to 180 degrees
- moved R4 139.9 mm to (163.4, 50.0)
- moved TP9 139.8 mm to (179.0, 67.5)
- moved R5 139.1 mm to (163.3, 45.6)
- moved TP1 136.8 mm to (175.5, 23.5)
- moved TP11 136.2 mm to (179.0, 58.0)
- moved R7 135.7 mm to (160.1, 50.0), turned to 180 degrees
- moved R18 128.1 mm to (147.0, 53.4), turned to -90 degrees
- moved R2 124.4 mm to (147.0, 47.1), turned to 90 degrees
- moved R17 117.0 mm to (134.5, 47.2), turned to 90 degrees
- moved R6 116.2 mm to (140.5, 36.9), turned to -90 degrees
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
Commit message: adjustments to layout
Parts:
- moved C4 63.4 mm to (72.8, 35.0), turned to 0 degrees
- moved R15 59.5 mm to (122.5, 21.4)
- moved TP9 53.6 mm to (164.0, 16.0)
- moved TP11 52.4 mm to (147.0, 16.5)
- moved R6 47.6 mm to (187.6, 30.0), turned to 180 degrees
- moved R1 45.3 mm to (177.0, 68.1), turned to 90 degrees
- moved R2 44.5 mm to (184.1, 22.5), turned to 180 degrees
- moved BT1 42.1 mm to (65.0, 18.3), turned to 180 degrees
- moved R8 38.2 mm to (161.0, 37.9), turned to -90 degrees
- moved R18 36.9 mm to (169.0, 83.1), turned to 90 degrees
- moved C1 36.8 mm to (168.0, 62.0), turned to -90 degrees
- moved R16 36.0 mm to (133.3, 43.5), turned to 0 degrees
- moved TP5 32.1 mm to (95.5, 80.5)
- moved R5 28.3 mm to (191.5, 47.9), turned to -90 degrees
- moved RV3 27.6 mm to (84.5, 27.5)
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
Commit message: adjustments
Parts:
- moved TP1 162.9 mm to (44.5, 71.5)
- moved TP3 144.9 mm to (60.5, 71.5)
- moved R2 144.2 mm to (40.0, 29.1), turned to 90 degrees
- moved R6 140.2 mm to (50.4, 59.0), turned to 0 degrees
- moved R3 139.2 mm to (60.5, 54.5), turned to 180 degrees
- moved R5 126.6 mm to (65.4, 36.5), turned to 0 degrees
- moved U1 124.8 mm to (55.5, 40.5), turned to 0 degrees
- moved C1 124.8 mm to (44.8, 42.5), turned to 0 degrees
- moved C2 116.8 mm to (44.8, 38.0), turned to 0 degrees
- moved R7 116.8 mm to (60.5, 63.5), turned to 180 degrees
- moved R1 114.9 mm to (65.4, 40.5), turned to 0 degrees
- moved R4 89.1 mm to (65.5, 44.5), turned to 0 degrees
- moved TP17 84.6 mm to (141.0, 62.0)
- moved TP9 72.1 mm to (120.5, 73.5)
- moved TP11 52.1 mm to (132.5, 66.5)
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
Commit message: finished routing
Parts:
- moved TP7 28.7 mm to (71.5, 66.5)
- moved TP5 28.0 mm to (64.0, 50.5)
- moved TP9 15.8 mm to (105.4, 68.6)
- moved TP3 12.8 mm to (65.0, 59.5)
- moved R6 12.5 mm to (59.6, 50.5), turned to 180 degrees
- moved R1 10.2 mm to (75.6, 40.5), turned to 180 degrees
- moved R7 9.05 mm to (59.6, 54.5)
- moved TP1 8.32 mm to (49.0, 64.5)
- moved R3 5.08 mm to (59.6, 59.5)
- moved TP8 4.00 mm to (129.6, 21.0)
- moved TP10 2.00 mm to (113.5, 20.0)
- moved TP6 2.00 mm to (104.5, 20.5)
- moved TP17 1.50 mm to (139.5, 62.0)
Routing:
- net GND: track 0.00 -> 314.4 mm
- net VCC: track 0.00 -> 142.9 mm, vias 0 -> 2
- net error_input: track 0.00 -> 110.2 mm, vias 0 -> 2
- net Vanode: track 0.00 -> 106.2 mm, vias 0 -> 2
- net Summing_Vn: track 0.00 -> 103.5 mm, vias 0 -> 8
- net Vcathode: track 0.00 -> 96.7 mm
- net Vset: track 0.00 -> 77.8 mm
- net D_Vn: track 0.00 -> 71.5 mm, vias 0 -> 1
- net I_Vn: track 0.00 -> 56.5 mm, vias 0 -> 6
- net P_Vn: track 0.00 -> 42.8 mm
- net Vcurr: track 0.00 -> 41.0 mm
- net error_output: track 0.00 -> 35.4 mm, vias 0 -> 4
- net BJT_Base: track 0.00 -> 34.9 mm
- net Net-(C7-Pad2): track 0.00 -> 32.1 mm
- net Net-(C6-Pad2): track 0.00 -> 30.7 mm
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Other:
- board outline added: 113.5 x 55.5 mm

Commit message: Finished PCb design, need to order pcb
Parts:
- moved TP8 11.1 mm to (119.4, 25.4)
- moved TP6 7.98 mm to (96.5, 20.3)
- moved TP10 6.83 mm to (106.7, 20.3)
- moved TP12 3.69 mm to (142.2, 30.5)
Routing:
- net D_Vn: track 71.5 -> 64.7 mm
- net BJT_Base: track 34.9 -> 31.1 mm
- net P_Vn: track 42.8 -> 44.6 mm
- net error_output: track 35.4 -> 34.6 mm
Other:
- board text added: "Analog PID Controller"
- board text added: "Devansh Joshi, Suren Shirani"
- board text added: "UT ECE - 03/07/2026"
Changed lines of the file:
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@@
 		(at 81.29 59.5 -90)
 		(property "Reference" "RV1"
-			(at 0 0 90)
+			(at -1.08 5.09 90)
 			(layer "F.SilkS")
 			(effects
@@
 		)
 		(property "Value" "TP_PID_error_input"
-			(at 8.47 1.25 0)
+			(at 9.66 2.84 0)
 			(layer "F.Fab")
 			(effects
@@
 		(tags "C Disc series Radial pin pitch 2.50mm diameter 3.8mm width 2.6mm Capacitor")
 		(property "Reference" "C1"
-			(at 1.25 0 0)
+			(at -1.57 -1.86 0)
 			(layer "F.SilkS")
 			(effects
@@
 		(tags "C Disc series Radial pin pitch 2.50mm diameter 3.8mm width 2.6mm Capacitor")
 		(property "Reference" "C2"
-			(at 1.25 0 0)
+			(at -1.57 -2.44 0)
 			(layer "F.SilkS")
 			(effects
@@
 		(tags "Through Hole Mount Test Points")
 		(property "Reference" "TP3"
-			(at 0 0 0)
+			(at 3.58 0 0)
 			(layer "F.SilkS")
 			(effects
@@
 	(footprint "TestPoint:TestPoint_Keystone_5010-5014_Multipurpose"
 		(layer "F.Cu")
-		(at 141 27)
+		(at 142.24 30.48)
 		(descr "Keystone THM Multipurpose Test Point 5010-5014, http://www.keyelco.com/product-pdf.cfm?p=1319")
 		(tags "Through Hole Mount Test Points")
@@
 		)
 		(property "Value" "TP_BJT_Base"
-			(at 0 0 0)
+			(at -5.08 0 90)
 			(layer "F.Fab")
 			(effects
@@
 	(footprint "TestPoint:TestPoint_Keystone_5010-5014_Multipurpose"
 		(layer "F.Cu")
-		(at 104.5 20.5)
+		(at 96.52 20.32)
 		(descr "Keystone THM Multipurpose Test Point 5010-5014, http://www.keyelco.com/product-pdf.cfm?p=1319")
 		(tags "Through Hole Mount Test Points")
 		(property "Reference" "TP6"
-			(at 0 -2.75 0)
+			(at 2.18 2.36 0)
 			(layer "F.SilkS")
 			(effects
@@
 		)
 		(property "Value" "TP_P_Vn_amp"
-			(at 0 2.75 0)
+			(at -2.9 -2.72 180)
 			(layer "F.Fab")
 			(effects
@@
 	(footprint "TestPoint:TestPoint_Keystone_5010-5014_Multipurpose"
 		(layer "F.Cu")
-		(at 129.56 21)
+		(at 119.38 25.4)
 		(descr "Keystone THM Multipurpose Test Point 5010-5014, http://www.keyelco.com/product-pdf.cfm?p=1319")
 		(tags "Through Hole Mount Test Points")
 		(property "Reference" "TP8"
-			(at 0 -2.75 0)
+			(at -5.08 -2.54 0)
 			(layer "F.SilkS")
 			(effects
@@
 		)
 		(property "Value" "TP_D_Vn_amp"
-			(at 8.47 1.25 0)
+			(at 7.62 0 0)
 			(layer "F.Fab")
 			(effects
@@
 	(footprint "TestPoint:TestPoint_Keystone_5010-5014_Multipurpose"
 		(layer "F.Cu")
-		(at 113.5 20)
+		(at 106.68 20.32)
 		(descr "Keystone THM Multipurpose Test Point 5010-5014, http://www.keyelco.com/product-pdf.cfm?p=1319")
 		(tags "Through Hole Mount Test Points")
 		(property "Reference" "TP10"
-			(at 0 -2.75 0)
+			(at 3.34 2.86 0)
 			(layer "F.SilkS")
 			(effects
@@
 		)
 		(property "Value" "TP_Error_output"
-			(at 0 2.75 0)
+			(at 0.8 -2.22 0)
 			(layer "F.Fab")
 			(effects
@@
 	)
 	(gr_rect
+		(start 121.92 16.03)
+		(end 144.78 23.65)
+		(stroke
+			(width 0.1)
+			(type default)
+		)
+		(fill no)
+		(layer "F.SilkS")
+	)
+	(gr_rect
 		(start 31.5 15.5)
 		(end 145 71)
@@
 		(layer "Edge.Cuts")
 	)
+	(gr_text "UT ECE - 03/07/2026"
+		(at 124.46 22.86 0)
+		(layer "F.SilkS")
+		(effects
+			(font
+				(size 1 1)
+				(thickness 0.1)
+			)
+			(justify left bottom)
+		)
+	)
+	(gr_text "Analog PID Controller"
+		(at 124.46 20.32 0)
+		(layer "F.SilkS")
+		(effects
+			(font
+				(size 1 1)
+				(thickness 0.1)
+			)
+			(justify left bottom)
+		)
+	)
+	(gr_text "Devansh Joshi, Suren Shirani"
+		(at 121.92 17.78 0)
+		(layer "F.SilkS")
+		(effects
+			(font
+				(size 1 1)
+				(thickness 0.1)
+			)
+			(justify left bottom)
+		)
+	)
 	(segment
 		(start 141 62)
@@
 	)
 	(segment
+		(start 121.92 27.94)
+		(end 119.38 25.4)
+		(width 0.2)
+		(layer "F.Cu")
+		(net 3)
+	)
+	(segment
 		(start 124.411 53.62605)
 		(end 124.411 52.04395)
@@
 	)
 	(segment
-		(start 110.787097 39.749953)
-		(end 110.410047 39.749953)
+		(start 121.911 51.399)
+		(end 120.81 52.5)
 		(width 0.2)
 		(layer "F.Cu")
@@
 	)
 	(segment
-		(start 129.56 20.97705)
-		(end 110.787097 39.749953)
+		(start 110.929225 39.609238)
+		(end 121.92 28.618463)
 		(width 0.2)
 		(layer "F.Cu")
@@
 	)
 	(segment
-		(start 121.911 51.399)
-		(end 120.81 52.5)
+		(start 121.92 28.618463)
+		(end 121.92 27.94)
 		(width 0.2)
 		(layer "F.Cu")
@@
 		(net 3)
 	)
+	(segment
+		(start 110.550762 39.609238)
+		(end 110.929225 39.609238)
+		(width 0.2)
+		(layer "F.Cu")
+		(net 3)
+	)
 	(via
 		(at 110.550762 39.609238)
@@
 	)
 	(segment
-		(start 104.5 27.44)
-		(end 104.5 20.5)
-		(width 0.2)
-		(layer "F.Cu")
-		(net 17)
-	)
-	(segment
 		(start 89.10395 37.521)
 		(end 88.306 36.72305)
@@
 	)
 	(segment
-		(start 104.56 27.5)
-		(end 104.5 27.44)
+		(start 102.446 29.614)
+		(end 101.56 30.5)
 		(width 0.2)
 		(layer "F.Cu")
@@
 	)
 	(segment
+		(start 96.52 20.32)
+		(end 102.446 26.246)
+		(width 0.2)
+		(layer "F.Cu")
+		(net 17)
+	)
+	(segment
 		(start 90.01605 37.521)
 		(end 89.10395 37.521)
@@
 	)
 	(segment
-		(start 101.56 30.5)
-		(end 104.56 27.5)
+		(start 102.446 26.246)
+		(end 102.446 29.614)
 		(width 0.2)
 		(layer "F.Cu")
@@
 	)
 	(segment
-		(start 121.06 33.92)
-		(end 117.58 33.92)
+		(start 106.68 20.32)
+		(end 106.68 25.14)
 		(width 0.2)
 		(layer "F.Cu")
@@
 	)
 	(segment
-		(start 113.56 23.9)
-		(end 113.5 23.84)
+		(start 121.06 33.92)
+		(end 117.58 33.92)
 		(width 0.2)
 		(layer "F.Cu")
@@
 	)
 	(segment
-		(start 113.5 23.84)
-		(end 113.5 20)
+		(start 106.68 25.14)
+		(end 109.5 27.96)
 		(width 0.2)
 		(layer "F.Cu")
@@
 	)
 	(segment
-		(start 113.56 23.9)
-		(end 109.5 27.96)
-		(width 0.2)
-		(layer "F.Cu")
-		(net 21)
-	)
-	(segment
 		(start 111 28.9)
 		(end 110.44 28.9)
@@
 	)
 	(segment
-		(start 142 28)
-		(end 141 27)
+		(start 142.24 36.32)
+		(end 140.56 38)
 		(width 0.2)
 		(layer "F.Cu")
@@
 	)
 	(segment
-		(start 142 36.56)
-		(end 142 28)
+		(start 122.161 42.979)
+		(end 121.06 44.08)
 		(width 0.2)
 		(layer "F.Cu")
@@
 	)
 	(segment
-		(start 122.161 42.979)
-		(end 121.06 44.08)
+		(start 142.24 30.48)
+		(end 142.24 36.32)
 		(width 0.2)
 		(layer "F.Cu")
@@
 		(width 0.2)
 		(layer "F.Cu")
-		(net 22)
-	)
-	(segment
-		(start 140.56 38)
-		(end 142 36.56)
-		(width 0.2)
-		(layer "F.Cu")
